File: hardware/kicad/Hidroponik_IoT_Cikidang.kicad_sch (KiCad schematic)
At the start: 33 parts, among them J1 ADS1115, J10 PUMP, J11 DC_IN_TERMINAL, J12 ESP_GPIO_LEFT, J13 ESP_GPIO_RIGHT, J2 DS18B20, J3 EC, J4 PH, J5 PUMP, J6 ADS_A2, J7 I2C, J8 ADS_A3, J9 Barrel_Jack_Switch, Q1 IRF520, Q2 IRF520, SW1 ESP_EN_JP, U1 ESP32-DevKitC

Commit message: Update Hidroponik_IoT_Cikidang.kicad_sch
Connections:
- net +3V3: now also R1.2, R3.2

Commit message: Update PCB Layout
Parts:
- J4: renamed from J11; footprint TerminalBlock_Phoenix:TerminalBlock_Phoenix_MPT-0,5-2-2.54_1x02_P2.54mm_Horizontal -> TerminalBlock_Phoenix:TerminalBlock_Phoenix_MKDS-1,5-2-5.08_1x02_P5.08mm_Horizontal
- renumbered C2 to C1, C1 to C2, C4 to C3, C3 to C4, D3 to D2, D2 to D3, J12 to J1, J3 to J10, J6 to J11, J8 to J12, J4 to J13, J13 to J2, J9 to J3, J10 to J6, J2 to J8, J1 to J9, Q2 to Q1, Q1 to Q2, R3 to R2, R4 to R3, R2 to R4, R6 to R5, R5 to R6
Connections:
- net +3V3: no longer R1.2, R2.2, R3.2
- net +5V: now also R1.2, R2.2, R3.2
- net ESP_GPIO12: now also R6.2; no longer R5.2
- net ESP_GPIO14: now also R5.2; no longer R6.2
