File: hardware/kicad/Hidroponik_IoT_Cikidang.kicad_pcb (KiCad board)
At the start: 2 copper layers, 81.5 x 58.7 mm, 31 parts, among them J1 ADS1115, J10 PUMP, J11 DC_IN_TERMINAL, J12 ESP_GPIO_LEFT, J13 ESP_GPIO_RIGHT, J2 DS18B20, J3 TDS, J4 TURBIDITY, J5 pH, J6 SERVO, J7 OLED, J9 Barrel_Jack_Switch, Q1 IRF520, SW1 ESP_EN_JP, U1 ESP32-DevKitC

Commit message: Update PCB Layout
Parts:
- removed the J6 at (47.0, 130.0)
- removed the R4 at (108.5, 113.8)
- removed REF** (x2): MountingHole_3.2mm_M3_DIN965_Pad, MountingHole:MountingHole_3.2mm_M3_DIN965_Pad
- added D2: IN4004, Diode_THT:D_DO-34_SOD68_P7.62mm_Horizontal, F.Cu at (116.7, 83.6)
- added J11: ADS_A2, Connector_Molex:Molex_SL_171971-0003_1x03_P2.54mm_Vertical, F.Cu at (182.4, 107.6)
- added J12: ADS_A3, Connector_Molex:Molex_SL_171971-0003_1x03_P2.54mm_Vertical, F.Cu at (177.3, 119.6)
- added Q1: IRF520, Package_TO_SOT_THT:TO-220-3_Vertical, F.Cu at (120.1, 84.8)
- added R2: 4.7k, Resistor_THT:R_Axial_DIN0204_L3.6mm_D1.6mm_P7.62mm_Horizontal, F.Cu at (172.0, 83.2)
- added R5: 1k, Resistor_THT:R_Axial_DIN0204_L3.6mm_D1.6mm_P7.62mm_Horizontal, F.Cu at (125.4, 83.6)
- J10: renamed from J3; value TDS -> EC
- J13: renamed from J4; value TURBIDITY -> PH
- J4: renamed from J11; footprint TerminalBlock_Phoenix:TerminalBlock_Phoenix_MPT-0,5-2-2.54_1x02_P2.54mm_Horizontal -> TerminalBlock_Phoenix:TerminalBlock_Phoenix_MKDS-1,5-2-5.08_1x02_P5.08mm_Horizontal
- J5: value pH -> PUMP; footprint Connector_Molex:Molex_SL_171971-0006_1x06_P2.54mm_Vertical -> Connector_Molex:Molex_SL_171971-0002_1x02_P2.54mm_Vertical
- J7: value OLED -> I2C
- moved R3 70.5 mm to (174.3, 83.2)
- moved C3 69.1 mm to (119.5, 108.5)
- moved D3 69.1 mm to (116.7, 103.9)
- moved C4 69.1 mm to (125.4, 108.5)
- moved Q2 69.1 mm to (120.1, 97.3)
- moved R4 69.1 mm to (118.3, 113.5)
- moved R6 69.1 mm to (125.4, 96.3)
- moved JP2 68.2 mm to (169.6, 86.6)
- moved C1 68.2 mm to (138.9, 121.8)
- moved C2 68.2 mm to (138.8, 76.6)
- moved J1 68.2 mm to (129.7, 76.4)
- moved J13 68.2 mm to (182.4, 95.9)
- moved J6 68.2 mm to (108.1, 108.6)
- moved J7 68.2 mm to (108.1, 88.3)
- moved SW1 68.2 mm to (108.1, 74.1)
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- renumbered C2 to C1, C1 to C2, C4 to C3, C3 to C4, D2 to D3, J12 to J1, J13 to J2, J9 to J3, J10 to J6, J2 to J8, J1 to J9, Q1 to Q2, R2 to R4, R5 to R6
Connections:
- net /PUMP_DIGITAL renamed /ESP_GPIO12
- net /PUMP_GND renamed /PUMP1_GND
- net /TDS_ANALOG renamed /EC_ANALOG
- J13 pad 1: /TURBIDITY_ANALOG -> /PH_ANALOG
- J5 pad 2: GND -> /PUMP2_GND
- J9 pad 8: /TURBIDITY_ANALOG -> /PH_ANALOG
- J9 pad 9: /PH_ANALOG -> /ADS1115_A2
- R1 pad 1: /DS18B20_DIGITAL -> /ADS1115_SDA
- R3 pad 1: /ADS1115_SCL -> /DS18B20_DIGITAL
Routing:
- net /ADS1115_A3: track 0.00 -> 30.5 mm
- net /ADS1115_A2: track 0.00 -> 26.2 mm
- net /ESP_GPIO25: track 26.7 -> 3.81 mm
- net /PUMP2_GND: track 0.00 -> 19.8 mm
- net /ESP_GPIO14: track 3.81 -> 20.8 mm
- net /TURBIDITY_ANALOG: track 16.6 -> 0.00 mm
- net /PH_ANALOG: track 32.6 -> 17.4 mm
- net +5V: track 237.9 -> 248.2 mm
- net /PUMP1_GND: track 17.8 -> 23.9 mm
- net Net-(D1-A): track 6.30 -> 12.1 mm
- net Net-(Q1-G): track 0.00 -> 5.79 mm
- net /ADS1115_SDA: track 72.4 -> 77.5 mm
- net /ESP_RESET: track 27.4 -> 29.4 mm
- net /ESP_GPIO12: track 8.80 -> 10.3 mm
- net /EC_ANALOG: track 21.3 -> 22.6 mm
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Other:
- board text added: "EC"
- board text added: "PUMP1"
- board text added: "PUMP2"
- board text removed: "Design Proyek - Konservasi Air"
- board text removed: "Kelompok 1.9 - Nov 2023"
- board text removed: "PUMP"
- board text removed: "PWM"
- board text removed: "SERVO"
- board text removed: "TDS"
- board text removed: "TURBIDITY"

Commit message: Update PCB
Parts:
- added ?: , , F.Cu at (118.0, 70.5)
- added REF**: MountingHole_3.2mm_M3_DIN965_Pad, MountingHole:MountingHole_3.2mm_M3_DIN965_Pad, F.Cu at (167.8, 119.5)
Routing:
- net /ADS1115_A3: track 30.5 -> 29.8 mm
- net GND: vias 0 -> 171
Other:
- board text added: "A2"
- board text added: "A3"
